File: smol-keypad.sch (KiCad schematic (older format))
At the start: 38 parts, among them SW1 SW_PUSH, U1 ProMicro

Commit message: night
Parts:
- removed H1, H2, H3, H4: MountingHole, MountingHole:MountingHole_2.2mm_M2, symbol Mechanical:MountingHole
- removed SW1: SW_PUSH, Button_Switch_SMD:SW_SPST_TL3342, symbol keyboard_parts:SW_PUSH
- added H1, H2, H3, H4: MountingHole_Pad, MountingHole:MountingHole_2.2mm_M2_Pad, symbol Mechanical:MountingHole_Pad
- MX1, MX10, MX11, MX12, MX13, MX14, MX15, MX16, MX2, MX3, MX4, MX5, MX6, MX7, MX8, MX9: footprint MX_Only:MXOnly-1U-NoLED -> keyswitches1U:Kailh_socket_MX
Connections:
- wire segments 59 -> 63
- no-connect marks 0 -> 13
Changed lines of the file:
@@
 F 0 "MX1" H 5133 1973 60  0000 C CNN
 F 1 "MX-NoLED" H 5133 1899 20  0000 C CNN
-F 2 "MX_Only:MXOnly-1U-NoLED" H 4475 1725 60  0001 C CNN
+F 2 "keyswitches1U:Kailh_socket_MX" H 4475 1725 60  0001 C CNN
 F 3 "" H 4475 1725 60  0001 C CNN
 	1    5100 1750
@@
 F 0 "MX2" H 5583 1973 60  0000 C CNN
 F 1 "MX-NoLED" H 5583 1899 20  0000 C CNN
-F 2 "MX_Only:MXOnly-1U-NoLED" H 4925 1725 60  0001 C CNN
+F 2 "keyswitches1U:Kailh_socket_MX" H 4925 1725 60  0001 C CNN
 F 3 "" H 4925 1725 60  0001 C CNN
 	1    5550 1750
@@
 F 0 "MX5" H 5133 2623 60  0000 C CNN
 F 1 "MX-NoLED" H 5133 2549 20  0000 C CNN
-F 2 "MX_Only:MXOnly-1U-NoLED" H 4475 2375 60  0001 C CNN
+F 2 "keyswitches1U:Kailh_socket_MX" H 4475 2375 60  0001 C CNN
 F 3 "" H 4475 2375 60  0001 C CNN
 	1    5100 2400
@@
 F 0 "MX6" H 5583 2623 60  0000 C CNN
 F 1 "MX-NoLED" H 5583 2549 20  0000 C CNN
-F 2 "MX_Only:MXOnly-1U-NoLED" H 4925 2375 60  0001 C CNN
+F 2 "keyswitches1U:Kailh_socket_MX" H 4925 2375 60  0001 C CNN
 F 3 "" H 4925 2375 60  0001 C CNN
 	1    5550 2400
@@
 F 0 "MX9" H 5133 3273 60  0000 C CNN
 F 1 "MX-NoLED" H 5133 3199 20  0000 C CNN
-F 2 "MX_Only:MXOnly-1U-NoLED" H 4475 3025 60  0001 C CNN
+F 2 "keyswitches1U:Kailh_socket_MX" H 4475 3025 60  0001 C CNN
 F 3 "" H 4475 3025 60  0001 C CNN
 	1    5100 3050
@@
 F 0 "MX10" H 5583 3273 60  0000 C CNN
 F 1 "MX-NoLED" H 5583 3199 20  0000 C CNN
-F 2 "MX_Only:MXOnly-1U-NoLED" H 4925 3025 60  0001 C CNN
+F 2 "keyswitches1U:Kailh_socket_MX" H 4925 3025 60  0001 C CNN
 F 3 "" H 4925 3025 60  0001 C CNN
 	1    5550 3050
@@
 F 0 "MX13" H 5133 3923 60  0000 C CNN
 F 1 "MX-NoLED" H 5133 3849 20  0000 C CNN
-F 2 "MX_Only:MXOnly-1U-NoLED" H 4475 3675 60  0001 C CNN
+F 2 "keyswitches1U:Kailh_socket_MX" H 4475 3675 60  0001 C CNN
 F 3 "" H 4475 3675 60  0001 C CNN
 	1    5100 3700
@@
 F 0 "MX14" H 5583 3923 60  0000 C CNN
 F 1 "MX-NoLED" H 5583 3849 20  0000 C CNN
-F 2 "MX_Only:MXOnly-1U-NoLED" H 4925 3675 60  0001 C CNN
+F 2 "keyswitches1U:Kailh_socket_MX" H 4925 3675 60  0001 C CNN
 F 3 "" H 4925 3675 60  0001 C CNN
 	1    5550 3700
@@
 F 0 "MX3" H 6033 1973 60  0000 C CNN
 F 1 "MX-NoLED" H 6033 1899 20  0000 C CNN
-F 2 "MX_Only:MXOnly-1U-NoLED" H 5375 1725 60  0001 C CNN
+F 2 "keyswitches1U:Kailh_socket_MX" H 5375 1725 60  0001 C CNN
 F 3 "" H 5375 1725 60  0001 C CNN
 	1    6000 1750
@@
 F 0 "MX4" H 6483 1973 60  0000 C CNN
 F 1 "MX-NoLED" H 6483 1899 20  0000 C CNN
-F 2 "MX_Only:MXOnly-1U-NoLED" H 5825 1725 60  0001 C CNN
+F 2 "keyswitches1U:Kailh_socket_MX" H 5825 1725 60  0001 C CNN
 F 3 "" H 5825 1725 60  0001 C CNN
 	1    6450 1750
@@
 F 0 "MX7" H 6033 2623 60  0000 C CNN
 F 1 "MX-NoLED" H 6033 2549 20  0000 C CNN
-F 2 "MX_Only:MXOnly-1U-NoLED" H 5375 2375 60  0001 C CNN
+F 2 "keyswitches1U:Kailh_socket_MX" H 5375 2375 60  0001 C CNN
 F 3 "" H 5375 2375 60  0001 C CNN
 	1    6000 2400
@@
 F 0 "MX8" H 6483 2623 60  0000 C CNN
 F 1 "MX-NoLED" H 6483 2549 20  0000 C CNN
-F 2 "MX_Only:MXOnly-1U-NoLED" H 5825 2375 60  0001 C CNN
+F 2 "keyswitches1U:Kailh_socket_MX" H 5825 2375 60  0001 C CNN
 F 3 "" H 5825 2375 60  0001 C CNN
 	1    6450 2400
@@
 F 0 "MX11" H 6033 3273 60  0000 C CNN
 F 1 "MX-NoLED" H 6033 3199 20  0000 C CNN
-F 2 "MX_Only:MXOnly-1U-NoLED" H 5375 3025 60  0001 C CNN
+F 2 "keyswitches1U:Kailh_socket_MX" H 5375 3025 60  0001 C CNN
 F 3 "" H 5375 3025 60  0001 C CNN
 	1    6000 3050
@@
 F 0 "MX12" H 6483 3273 60  0000 C CNN
 F 1 "MX-NoLED" H 6483 3199 20  0000 C CNN
-F 2 "MX_Only:MXOnly-1U-NoLED" H 5825 3025 60  0001 C CNN
+F 2 "keyswitches1U:Kailh_socket_MX" H 5825 3025 60  0001 C CNN
 F 3 "" H 5825 3025 60  0001 C CNN
 	1    6450 3050
@@
 F 0 "MX15" H 6033 3923 60  0000 C CNN
 F 1 "MX-NoLED" H 6033 3849 20  0000 C CNN
-F 2 "MX_Only:MXOnly-1U-NoLED" H 5375 3675 60  0001 C CNN
+F 2 "keyswitches1U:Kailh_socket_MX" H 5375 3675 60  0001 C CNN
 F 3 "" H 5375 3675 60  0001 C CNN
 	1    6000 3700
@@
 F 0 "MX16" H 6483 3923 60  0000 C CNN
 F 1 "MX-NoLED" H 6483 3849 20  0000 C CNN
-F 2 "MX_Only:MXOnly-1U-NoLED" H 5825 3675 60  0001 C CNN
+F 2 "keyswitches1U:Kailh_socket_MX" H 5825 3675 60  0001 C CNN
 F 3 "" H 5825 3675 60  0001 C CNN
 	1    6450 3700
@@
 	0    -1   -1   0
 $EndComp
-Wire Wire Line
-	2550 1350 3050 1350
-$Comp
-L keyboard_parts:SW_PUSH SW1
-U 1 1 61AD0DE1
-P 3350 1350
-F 0 "SW1" H 3350 1605 50  0000 C CNN
-F 1 "SW_PUSH" H 3350 1514 50  0000 C CNN
-F 2 "Button_Switch_SMD:SW_SPST_TL3342" H 3350 1350 60  0001 C CNN
-F 3 "" H 3350 1350 60  0000 C CNN
-	1    3350 1350
-	1    0    0    -1
-$EndComp
-$Comp
-L power:GND #PWR0102
-U 1 1 61AD1703
-P 3800 1350
-F 0 "#PWR0102" H 3800 1100 50  0001 C CNN
-F 1 "GND" V 3805 1222 50  0000 R CNN
-F 2 "" H 3800 1350 50  0001 C CNN
-F 3 "" H 3800 1350 50  0001 C CNN
-	1    3800 1350
-	0    -1   -1   0
-$EndComp
-Wire Wire Line
-	3650 1350 3800 1350
 Text Label 4500 2100 0    50   ~ 0
 row0
@@
 Text Label 6600 1050 0    50   ~ 0
 col3
-$Comp
-L Mechanical:MountingHole H1
-U 1 1 60A654B7
-P 1300 2800
-F 0 "H1" H 1400 2846 50  0000 L CNN
-F 1 "MountingHole" H 1400 2755 50  0000 L CNN
-F 2 "MountingHole:MountingHole_2.2mm_M2" H 1300 2800 50  0001 C CNN
-F 3 "~" H 1300 2800 50  0001 C CNN
-	1    1300 2800
-	1    0    0    -1
-$EndComp
-$Comp
-L Mechanical:MountingHole H2
-U 1 1 60A66FD9
-P 1300 3000
-F 0 "H2" H 1400 3046 50  0000 L CNN
-F 1 "MountingHole" H 1400 2955 50  0000 L CNN
-F 2 "MountingHole:MountingHole_2.2mm_M2" H 1300 3000 50  0001 C CNN
-F 3 "~" H 1300 3000 50  0001 C CNN
-	1    1300 3000
-	1    0    0    -1
-$EndComp
-$Comp
-L Mechanical:MountingHole H3
-U 1 1 60A6727E
-P 1300 3200
-F 0 "H3" H 1400 3246 50  0000 L CNN
-F 1 "MountingHole" H 1400 3155 50  0000 L CNN
-F 2 "MountingHole:MountingHole_2.2mm_M2" H 1300 3200 50  0001 C CNN
-F 3 "~" H 1300 3200 50  0001 C CNN
-	1    1300 3200
-	1    0    0    -1
-$EndComp
-$Comp
-L Mechanical:MountingHole H4
-U 1 1 60A67B53
-P 1300 3400
-F 0 "H4" H 1400 3446 50  0000 L CNN
-F 1 "MountingHole" H 1400 3355 50  0000 L CNN
-F 2 "MountingHole:MountingHole_2.2mm_M2" H 1300 3400 50  0001 C CNN
-F 3 "~" H 1300 3400 50  0001 C CNN
-	1    1300 3400
-	1    0    0    -1
-$EndComp
 Text Label 900  2250 0    50   ~ 0
 row3
@@
 Wire Wire Line
 	1150 1850 900  1850
+Wire Wire Line
+	1150 1350 900  1350
+Wire Wire Line
+	1150 1450 900  1450
+$Comp
+L power:GND #PWR0102
+U 1 1 60A9DA5A
+P 900 1350
+F 0 "#PWR0102" H 900 1100 50  0001 C CNN
+F 1 "GND" V 905 1222 50  0000 R CNN
+F 2 "" H 900 1350 50  0001 C CNN
+F 3 "" H 900 1350 50  0001 C CNN
+	1    900  1350
+	0    1    1    0
+$EndComp
+$Comp
+L power:GND #PWR0103
+U 1 1 60A9E836
+P 900 1450
+F 0 "#PWR0103" H 900 1200 50  0001 C CNN
+F 1 "GND" V 905 1322 50  0000 R CNN
+F 2 "" H 900 1450 50  0001 C CNN
+F 3 "" H 900 1450 50  0001 C CNN
+	1    900  1450
+	0    1    1    0
+$EndComp
+NoConn ~ 1150 1150
+NoConn ~ 1150 1250
+NoConn ~ 2550 1150
+NoConn ~ 2550 1350
+NoConn ~ 2550 1450
+NoConn ~ 2550 1550
+NoConn ~ 2550 1650
+NoConn ~ 2550 1750
+NoConn ~ 2550 1850
+NoConn ~ 2550 1950
+NoConn ~ 2550 2050
+NoConn ~ 2550 2150
+NoConn ~ 2550 2250
+$Comp
+L Mechanical:MountingHole_Pad H2
+U 1 1 60AAE5B6
+P 800 3350
+F 0 "H2" H 900 3399 50  0000 L CNN
+F 1 "MountingHole_Pad" H 900 3308 50  0000 L CNN
+F 2 "MountingHole:MountingHole_2.2mm_M2_Pad" H 800 3350 50  0001 C CNN
+F 3 "~" H 800 3350 50  0001 C CNN
+	1    800  3350
+	1    0    0    -1
+$EndComp
+$Comp
+L power:GND #PWR0104
+U 1 1 60AB94B2
+P 800 3600
+F 0 "#PWR0104" H 800 3350 50  0001 C CNN
+F 1 "GND" V 805 3472 50  0000 R CNN
+F 2 "" H 800 3600 50  0001 C CNN
+F 3 "" H 800 3600 50  0001 C CNN
+	1    800  3600
+	1    0    0    -1
+$EndComp
+Wire Wire Line
+	800  3450 800  3600
+$Comp
+L Mechanical:MountingHole_Pad H1
+U 1 1 60AC6A81
+P 800 2650
+F 0 "H1" H 900 2699 50  0000 L CNN
+F 1 "MountingHole_Pad" H 900 2608 50  0000 L CNN
+F 2 "MountingHole:MountingHole_2.2mm_M2_Pad" H 800 2650 50  0001 C CNN
+F 3 "~" H 800 2650 50  0001 C CNN
+	1    800  2650
+	1    0    0    -1
+$EndComp
+$Comp
+L power:GND #PWR0105
+U 1 1 60AC6A87
+P 800 2900
+F 0 "#PWR0105" H 800 2650 50  0001 C CNN
+F 1 "GND" V 805 2772 50  0000 R CNN
+F 2 "" H 800 2900 50  0001 C CNN
+F 3 "" H 800 2900 50  0001 C CNN
+	1    800  2900
+	1    0    0    -1
+$EndComp
+Wire Wire Line
+	800  2750 800  2900
+$Comp
+L Mechanical:MountingHole_Pad H3
+U 1 1 60AC8526
+P 2000 2700
+F 0 "H3" H 2100 2749 50  0000 L CNN
+F 1 "MountingHole_Pad" H 2100 2658 50  0000 L CNN
+F 2 "MountingHole:MountingHole_2.2mm_M2_Pad" H 2000 2700 50  0001 C CNN
+F 3 "~" H 2000 2700 50  0001 C CNN
+	1    2000 2700
+	1    0    0    -1
+$EndComp
+$Comp
+L power:GND #PWR0106
+U 1 1 60AC852C
+P 2000 2950
+F 0 "#PWR0106" H 2000 2700 50  0001 C CNN
+F 1 "GND" V 2005 2822 50  0000 R CNN
+F 2 "" H 2000 2950 50  0001 C CNN
+F 3 "" H 2000 2950 50  0001 C CNN
+	1    2000 2950
+	1    0    0    -1
+$EndComp
+Wire Wire Line
+	2000 2800 2000 2950
+$Comp
+L Mechanical:MountingHole_Pad H4
+U 1 1 60ACAC15
+P 2000 3450
+F 0 "H4" H 2100 3499 50  0000 L CNN
+F 1 "MountingHole_Pad" H 2100 3408 50  0000 L CNN
+F 2 "MountingHole:MountingHole_2.2mm_M2_Pad" H 2000 3450 50  0001 C CNN
+F 3 "~" H 2000 3450 50  0001 C CNN
+	1    2000 3450
+	1    0    0    -1
+$EndComp
+$Comp
+L power:GND #PWR0107
+U 1 1 60ACAC1B
+P 2000 3700
+F 0 "#PWR0107" H 2000 3450 50  0001 C CNN
+F 1 "GND" V 2005 3572 50  0000 R CNN
+F 2 "" H 2000 3700 50  0001 C CNN
+F 3 "" H 2000 3700 50  0001 C CNN
+	1    2000 3700
+	1    0    0    -1
+$EndComp
+Wire Wire Line
+	2000 3550 2000 3700
 $EndSCHEMATC

Commit message: add rotary encoders
Parts:
- added D17: D_Small, Diode_SMD:D_SOD-123, symbol Device:D_Small
- added SW1: Rotary_Encoder_Switch, Rotary_Encoder:RotaryEncoder_Alps_EC11E-Switch_Vertical_H20mm, symbol Device:Rotary_Encoder_Switch
Connections:
- net GND: now also SW1.C
- net row3: now also D17.1 (K)
- net pinA: now reaches U1.19 (F5)
- net pinA: now also SW1.A
- net pinB: now reaches U1.20 (F4)
- net pinB: now also SW1.B
- new net colRotEnc: SW1.S1
- new net rotEnc: D17.2 (A), SW1.S2
- no-connect marks 13 -> 10
Other:
- moved on the sheet: D1, D10, D11, D12, D13, D14, D15, D16, D2, D3, D4, D5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
