File: smol-keypad.sch (KiCad schematic (older format))
At the start: 40 parts, among them SW1 Rotary_Encoder_Switch, U1 ProMicro, U2 OLED

Commit message: final
Parts:
- removed U2: OLED, Display:Adafruit_SSD1306, symbol SSD1306-128x64_OLED:OLED
- added OL1: OLED, kbd:OLED_v2, symbol kbd:OLED
Connections:
- net GND: now also OL1.4 (GND)
- net SCL: now also U1.5 (SCL), OL1.2 (SCL)
- net SDA: now also U1.6 (SDA), OL1.1 (SDA)
- net VCC: now also OL1.3 (VCC)
- net col2: now also U1.13 (B6); no longer U1.6 (SDA)
- net col3: now also U1.14 (B2); no longer U1.5 (SCL)
- net colRotEnc: now also U1.15 (B3)
- no-connect marks 9 -> 7
Changed lines of the file:
@@
 $EndDescr
-$Comp
-L promicro:ProMicro U1
-U 1 1 61A526B2
-P 1850 1900
-F 0 "U1" H 1850 2937 60  0000 C CNN
-F 1 "ProMicro" H 1850 2831 60  0000 C CNN
-F 2 "promicro:ProMicro" H 1950 850 60  0001 C CNN
-F 3 "" H 1950 850 60  0000 C CNN
-	1    1850 1900
-	1    0    0    -1
-$EndComp
 $Comp
 L MX_Alps_Hybrid:MX-NoLED MX1
@@
 Wire Wire Line
 	5600 2800 5150 2800
-Connection ~ 5150 2800
 Wire Wire Line
 	5600 3450 5150 3450
-Connection ~ 5150 3450
 Wire Wire Line
 	5450 3050 5450 2400
@@
 Wire Wire Line
 	5900 2400 5900 1750
-Wire Wire Line
-	4700 3450 5150 3450
-Wire Wire Line
-	4700 2800 5150 2800
 $Comp
 L MX_Alps_Hybrid:MX-NoLED MX9
@@
 Wire Wire Line
 	5600 4100 5150 4100
-Connection ~ 5150 4100
 Wire Wire Line
 	5600 4750 5150 4750
@@
 Wire Wire Line
 	4700 4750 5150 4750
-Wire Wire Line
-	4700 4100 5150 4100
 $Comp
 L MX_Alps_Hybrid:MX-NoLED MX3
@@
 	0    -1   -1   0
 $EndComp
-Text Label 4700 2800 0    50   ~ 0
-row0
-Text Label 4700 3450 0    50   ~ 0
-row1
-Text Label 4700 4100 0    50   ~ 0
-row2
-Text Label 5450 1750 0    50   ~ 0
-col0
-Text Label 5900 1750 0    50   ~ 0
-col1
-Text Label 6350 1750 0    50   ~ 0
-col2
-Text Label 6800 1750 0    50   ~ 0
-col3
 Text Label 900  2250 0    50   ~ 0
 row3
@@
 Text Label 900  1750 0    50   ~ 0
 col1
-Text Label 900  1650 0    50   ~ 0
-col2
-Text Label 900  1550 0    50   ~ 0
-col3
-Wire Wire Line
-	900  1550 1150 1550
-Wire Wire Line
-	1150 1650 900  1650
 Wire Wire Line
 	900  1750 1150 1750
@@
 NoConn ~ 2550 1850
 NoConn ~ 2550 1950
-NoConn ~ 2550 2050
-NoConn ~ 2550 2150
 $Comp
 L Mechanical:MountingHole_Pad H2
@@
 	0    -1   -1   0
 $EndComp
-Wire Wire Line
-	1550 3350 1350 3350
-Wire Wire Line
-	1550 3550 1350 3550
-Text Label 1350 3550 0    50   ~ 0
-pinB
-Text Label 1350 3350 0    50   ~ 0
-pinA
-Wire Wire Line
-	1550 3450 1350 3450
+Text Label 4300 4750 0    50   ~ 0
+row3
+Connection ~ 4700 4750
+Wire Wire Line
+	4300 4750 4700 4750
+Wire Wire Line
+	2550 1450 2700 1450
+Text Label 2700 1450 0    50   ~ 0
+VCC
+$Comp
+L kbd:OLED OL1
+U 1 1 60C4879E
+P 2200 4800
+F 0 "OL1" H 2828 4869 51  0000 L CNN
+F 1 "OLED" H 2828 4779 47  0000 L CNN
+F 2 "kbd:OLED_v2" H 2200 4900 60  0001 C CNN
+F 3 "" H 2200 4900 60  0001 C CNN
+	1    2200 4800
+	1    0    0    -1
+$EndComp
+Text Label 2700 2150 0    50   ~ 0
+col3
+Text Label 2700 2250 0    50   ~ 0
+col2
+Text Label 6800 1750 0    50   ~ 0
+col3
+Text Label 6350 1750 0    50   ~ 0
+col2
+Text Label 5900 1750 0    50   ~ 0
+col1
+Text Label 5450 1750 0    50   ~ 0
+col0
+Wire Wire Line
+	4700 4550 4700 4400
+Wire Wire Line
+	2150 3350 2400 3350
+Text Label 2300 3550 0    50   ~ 0
+rotEnc
+Wire Wire Line
+	2150 3550 2300 3550
+$Comp
+L Device:Rotary_Encoder_Switch SW1
+U 1 1 60B0022B
+P 1850 3450
+F 0 "SW1" H 1850 3817 50  0000 C CNN
+F 1 "Rotary_Encoder_Switch" H 1850 3726 50  0000 C CNN
+F 2 "Keebio-Parts:RotaryEncoder_EC11" H 1700 3610 50  0001 C CNN
+F 3 "~" H 1850 3710 50  0001 C CNN
+	1    1850 3450
+	1    0    0    -1
+$EndComp
 $Comp
 L power:GND #PWR0108
@@
 	0    1    1    0
 $EndComp
-$Comp
-L Device:Rotary_Encoder_Switch SW1
-U 1 1 60B0022B
-P 1850 3450
-F 0 "SW1" H 1850 3817 50  0000 C CNN
-F 1 "Rotary_Encoder_Switch" H 1850 3726 50  0000 C CNN
-F 2 "Keebio-Parts:RotaryEncoder_EC11" H 1700 3610 50  0001 C CNN
-F 3 "~" H 1850 3710 50  0001 C CNN
-	1    1850 3450
-	1    0    0    -1
-$EndComp
-Text Label 4300 4750 0    50   ~ 0
-row3
-Connection ~ 4700 4750
-Wire Wire Line
-	4300 4750 4700 4750
-Wire Wire Line
-	4700 4550 4700 4400
-Text Label 4850 4400 0    50   ~ 0
-rotEnc
-Wire Wire Line
-	4700 4400 4850 4400
-Wire Wire Line
-	2150 3550 2300 3550
-Text Label 2300 3550 0    50   ~ 0
-rotEnc
-Wire Wire Line
-	2150 3350 2400 3350
+Wire Wire Line
+	1550 3450 1350 3450
+Text Label 1350 3350 0    50   ~ 0
+pinA
+Text Label 1350 3550 0    50   ~ 0
+pinB
+Wire Wire Line
+	1550 3550 1350 3550
+Wire Wire Line
+	1550 3350 1350 3350
 Wire Wire Line
 	2400 3350 2400 3050
 Text Label 2400 3050 0    50   ~ 0
 colRotEnc
-Text Label 2700 2250 0    50   ~ 0
+Wire Wire Line
+	4700 4400 4850 4400
+Text Label 4850 4400 0    50   ~ 0
+rotEnc
+Text Label 1200 4850 0    50   ~ 0
+VCC
+Wire Wire Line
+	1200 4850 1450 4850
+$Comp
+L power:GND #PWR0109
+U 1 1 60C4BC90
+P 1200 5000
+F 0 "#PWR0109" H 1200 4750 50  0001 C CNN
+F 1 "GND" V 1205 4872 50  0000 R CNN
+F 2 "" H 1200 5000 50  0001 C CNN
+F 3 "" H 1200 5000 50  0001 C CNN
+	1    1200 5000
+	0    1    1    0
+$EndComp
+Wire Wire Line
+	1450 5000 1200 5000
+Wire Wire Line
+	1450 4700 1200 4700
+Wire Wire Line
+	1450 4550 1200 4550
+Text Label 1200 4550 0    50   ~ 0
+SDA
+Text Label 1200 4700 0    50   ~ 0
+SCL
+Connection ~ 5150 4100
+Connection ~ 5150 3450
+Connection ~ 5150 2800
+Text Label 4700 4100 0    50   ~ 0
+row2
+Text Label 4700 3450 0    50   ~ 0
+row1
+Text Label 4700 2800 0    50   ~ 0
+row0
+Wire Wire Line
+	4700 4100 5150 4100
+Wire Wire Line
+	4700 2800 5150 2800
+Wire Wire Line
+	4700 3450 5150 3450
+Wire Wire Line
+	1150 1550 900  1550
+Wire Wire Line
+	1150 1650 900  1650
+Text Label 900  1650 0    50   ~ 0
+SDA
+Text Label 900  1550 0    50   ~ 0
+SCL
+Wire Wire Line
+	2700 2150 2550 2150
+Wire Wire Line
+	2700 2250 2550 2250
+$Comp
+L promicro:ProMicro U1
+U 1 1 61A526B2
+P 1850 1900
+F 0 "U1" H 1850 2937 60  0000 C CNN
+F 1 "ProMicro" H 1850 2831 60  0000 C CNN
+F 2 "promicro:ProMicro" H 1950 850 60  0001 C CNN
+F 3 "" H 1950 850 60  0000 C CNN
+	1    1850 1900
+	1    0    0    -1
+$EndComp
+Text Label 2700 2050 0    50   ~ 0
 colRotEnc
-$Comp
-L SSD1306-128x64_OLED:OLED U2
-U 1 1 60C2E002
-P 1650 4700
-F 0 "U2" H 1928 4804 50  0000 L CNN
-F 1 "OLED" H 1928 4713 50  0000 L CNN
-F 2 "Display:Adafruit_SSD1306" H 1650 4950 50  0001 C CNN
-F 3 "" H 1650 4950 50  0001 C CNN
-	1    1650 4700
-	0    1    1    0
-$EndComp
-$Comp
-L power:GND #PWR0109
-U 1 1 60C318F9
-P 2150 4550
-F 0 "#PWR0109" H 2150 4300 50  0001 C CNN
-F 1 "GND" V 2155 4422 50  0000 R CNN
-F 2 "" H 2150 4550 50  0001 C CNN
-F 3 "" H 2150 4550 50  0001 C CNN
-	1    2150 4550
-	0    -1   -1   0
-$EndComp
-Wire Wire Line
-	2000 4550 2150 4550
-Wire Wire Line
-	2550 1450 2700 1450
-Text Label 2700 1450 0    50   ~ 0
-VCC
-Text Label 2250 4650 0    50   ~ 0
-VCC
-Wire Wire Line
-	2000 4650 2250 4650
-Text Label 2250 4750 0    50   ~ 0
-SCL
-Text Label 2250 4850 0    50   ~ 0
-SDA
-Wire Wire Line
-	2000 4750 2250 4750
-Wire Wire Line
-	2250 4850 2000 4850
+Wire Wire Line
+	2550 2050 2700 2050
 $EndSCHEMATC

Commit message: update diode footprint
Parts:
- D1, D10, D11, D12, D13, D14, D15, D16, D17, D2, D3, D4, D5, D6, D7, D8, D9: footprint Diode_SMD:D_SOD-123 -> kbd:D3_TH_SMD_v2
Changed lines of the file:
@@
 F 0 "D1" V 5196 2630 50  0000 R CNN
 F 1 "D_Small" V 5105 2630 50  0000 R CNN
-F 2 "Diode_SMD:D_SOD-123" V 5150 2700 50  0001 C CNN
+F 2 "kbd:D3_TH_SMD_v2" V 5150 2700 50  0001 C CNN
 F 3 "~" V 5150 2700 50  0001 C CNN
 	1    5150 2700
@@
 F 0 "D2" V 5646 2630 50  0000 R CNN
 F 1 "D_Small" V 5555 2630 50  0000 R CNN
-F 2 "Diode_SMD:D_SOD-123" V 5600 2700 50  0001 C CNN
+F 2 "kbd:D3_TH_SMD_v2" V 5600 2700 50  0001 C CNN
 F 3 "~" V 5600 2700 50  0001 C CNN
 	1    5600 2700
@@
 F 0 "D5" V 5196 3280 50  0000 R CNN
 F 1 "D_Small" V 5105 3280 50  0000 R CNN
-F 2 "Diode_SMD:D_SOD-123" V 5150 3350 50  0001 C CNN
+F 2 "kbd:D3_TH_SMD_v2" V 5150 3350 50  0001 C CNN
 F 3 "~" V 5150 3350 50  0001 C CNN
 	1    5150 3350
@@
 F 0 "D6" V 5646 3280 50  0000 R CNN
 F 1 "D_Small" V 5555 3280 50  0000 R CNN
-F 2 "Diode_SMD:D_SOD-123" V 5600 3350 50  0001 C CNN
+F 2 "kbd:D3_TH_SMD_v2" V 5600 3350 50  0001 C CNN
 F 3 "~" V 5600 3350 50  0001 C CNN
 	1    5600 3350
@@
 F 0 "D9" V 5196 3930 50  0000 R CNN
 F 1 "D_Small" V 5105 3930 50  0000 R CNN
-F 2 "Diode_SMD:D_SOD-123" V 5150 4000 50  0001 C CNN
+F 2 "kbd:D3_TH_SMD_v2" V 5150 4000 50  0001 C CNN
 F 3 "~" V 5150 4000 50  0001 C CNN
 	1    5150 4000
@@
 F 0 "D10" V 5646 3930 50  0000 R CNN
 F 1 "D_Small" V 5555 3930 50  0000 R CNN
-F 2 "Diode_SMD:D_SOD-123" V 5600 4000 50  0001 C CNN
+F 2 "kbd:D3_TH_SMD_v2" V 5600 4000 50  0001 C CNN
 F 3 "~" V 5600 4000 50  0001 C CNN
 	1    5600 4000
@@
 F 0 "D13" V 5196 4580 50  0000 R CNN
 F 1 "D_Small" V 5105 4580 50  0000 R CNN
-F 2 "Diode_SMD:D_SOD-123" V 5150 4650 50  0001 C CNN
+F 2 "kbd:D3_TH_SMD_v2" V 5150 4650 50  0001 C CNN
 F 3 "~" V 5150 4650 50  0001 C CNN
 	1    5150 4650
@@
 F 0 "D14" V 5646 4580 50  0000 R CNN
 F 1 "D_Small" V 5555 4580 50  0000 R CNN
-F 2 "Diode_SMD:D_SOD-123" V 5600 4650 50  0001 C CNN
+F 2 "kbd:D3_TH_SMD_v2" V 5600 4650 50  0001 C CNN
 F 3 "~" V 5600 4650 50  0001 C CNN
 	1    5600 4650
@@
 F 0 "D3" V 6096 2630 50  0000 R CNN
 F 1 "D_Small" V 6005 2630 50  0000 R CNN
-F 2 "Diode_SMD:D_SOD-123" V 6050 2700 50  0001 C CNN
+F 2 "kbd:D3_TH_SMD_v2" V 6050 2700 50  0001 C CNN
 F 3 "~" V 6050 2700 50  0001 C CNN
 	1    6050 2700
@@
 F 0 "D4" V 6546 2630 50  0000 R CNN
 F 1 "D_Small" V 6455 2630 50  0000 R CNN
-F 2 "Diode_SMD:D_SOD-123" V 6500 2700 50  0001 C CNN
+F 2 "kbd:D3_TH_SMD_v2" V 6500 2700 50  0001 C CNN
 F 3 "~" V 6500 2700 50  0001 C CNN
 	1    6500 2700
@@
 F 0 "D7" V 6096 3280 50  0000 R CNN
 F 1 "D_Small" V 6005 3280 50  0000 R CNN
-F 2 "Diode_SMD:D_SOD-123" V 6050 3350 50  0001 C CNN
+F 2 "kbd:D3_TH_SMD_v2" V 6050 3350 50  0001 C CNN
 F 3 "~" V 6050 3350 50  0001 C CNN
 	1    6050 3350
@@
 F 0 "D8" V 6546 3280 50  0000 R CNN
 F 1 "D_Small" V 6455 3280 50  0000 R CNN
-F 2 "Diode_SMD:D_SOD-123" V 6500 3350 50  0001 C CNN
+F 2 "kbd:D3_TH_SMD_v2" V 6500 3350 50  0001 C CNN
 F 3 "~" V 6500 3350 50  0001 C CNN
 	1    6500 3350
@@
 F 0 "D11" V 6096 3930 50  0000 R CNN
 F 1 "D_Small" V 6005 3930 50  0000 R CNN
-F 2 "Diode_SMD:D_SOD-123" V 6050 4000 50  0001 C CNN
+F 2 "kbd:D3_TH_SMD_v2" V 6050 4000 50  0001 C CNN
 F 3 "~" V 6050 4000 50  0001 C CNN
 	1    6050 4000
@@
 F 0 "D12" V 6546 3930 50  0000 R CNN
 F 1 "D_Small" V 6455 3930 50  0000 R CNN
-F 2 "Diode_SMD:D_SOD-123" V 6500 4000 50  0001 C CNN
+F 2 "kbd:D3_TH_SMD_v2" V 6500 4000 50  0001 C CNN
 F 3 "~" V 6500 4000 50  0001 C CNN
 	1    6500 4000
@@
 F 0 "D15" V 6096 4580 50  0000 R CNN
 F 1 "D_Small" V 6005 4580 50  0000 R CNN
-F 2 "Diode_SMD:D_SOD-123" V 6050 4650 50  0001 C CNN
+F 2 "kbd:D3_TH_SMD_v2" V 6050 4650 50  0001 C CNN
 F 3 "~" V 6050 4650 50  0001 C CNN
 	1    6050 4650
@@
 F 0 "D16" V 6546 4580 50  0000 R CNN
 F 1 "D_Small" V 6455 4580 50  0000 R CNN
-F 2 "Diode_SMD:D_SOD-123" V 6500 4650 50  0001 C CNN
+F 2 "kbd:D3_TH_SMD_v2" V 6500 4650 50  0001 C CNN
 F 3 "~" V 6500 4650 50  0001 C CNN
 	1    6500 4650
@@
 F 0 "D17" V 4746 4580 50  0000 R CNN
 F 1 "D_Small" V 4655 4580 50  0000 R CNN
-F 2 "Diode_SMD:D_SOD-123" V 4700 4650 50  0001 C CNN
+F 2 "kbd:D3_TH_SMD_v2" V 4700 4650 50  0001 C CNN
 F 3 "~" V 4700 4650 50  0001 C CNN
 	1    4700 4650
