File: _autosave-smol-keypad.kicad_pcb (KiCad board)
At the start: 2 copper layers, 79.4 x 107.9 mm, 37 parts, among them U1 ProMicro

Commit message: night
Parts:
- moved U1 10.7 mm to (152.4, 42.9)
Routing:
- net /col3: track 83.1 -> 72.2 mm
- net /row2: track 131.7 -> 141.3 mm
- net /row1: track 114.4 -> 124.0 mm
- net /row0: track 97.6 -> 107.2 mm
- net /row3: track 148.7 -> 158.3 mm
- net /col0: track 93.1 -> 101.8 mm
- net /col1: track 78.7 -> 85.3 mm
- net /col2: track 70.8 -> 70.2 mm
Changed lines of the file:
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@@
     (thickness 1.6)
     (drawings 9)
-    (tracks 258)
+    (tracks 260)
     (zones 0)
     (modules 37)
@@
     )
   )
-  (module promicro:ProMicro (layer B.Cu)
-    (at 142.279568 39.290592 180)
+  (module promicro:ProMicro locked (layer B.Cu)
+    (at 152.399872 42.862464 180)
     (descr "Pro Micro footprint")
     (tags "promicro ProMicro")
@@
   (segment (start 112.650038 64.157626) (end 113.10928 63.698384) (width 0.25) (layer B.Cu) (net 2))
   (segment (start 110.331216 64.157626) (end 112.650038 64.157626) (width 0.25) (layer B.Cu) (net 2))
-  (segment (start 113.10928 61.79106) (end 121.917572 52.982768) (width 0.25) (layer F.Cu) (net 2))
-  (segment (start 113.10928 63.698384) (end 113.10928 61.79106) (width 0.25) (layer F.Cu) (net 2))
-  (segment (start 129.857392 52.982768) (end 135.929568 46.910592) (width 0.25) (layer F.Cu) (net 2))
-  (segment (start 121.917572 52.982768) (end 129.857392 52.982768) (width 0.25) (layer F.Cu) (net 2))
+  (segment (start 141.763632 54.768704) (end 146.049872 50.482464) (width 0.25) (layer F.Cu) (net 2))
+  (segment (start 113.10928 60.126512) (end 118.467088 54.768704) (width 0.25) (layer F.Cu) (net 2))
+  (segment (start 118.467088 54.768704) (end 141.763632 54.768704) (width 0.25) (layer F.Cu) (net 2))
+  (segment (start 113.10928 63.698384) (end 113.10928 60.126512) (width 0.25) (layer F.Cu) (net 2))
   (segment (start 115.708717 58.142625) (end 115.708717 58.122387) (width 0.25) (layer B.Cu) (net 3))
   (segment (start 113.883716 59.967626) (end 115.708717 58.142625) (width 0.25) (layer B.Cu) (net 3))
@@
   (segment (start 112.05471 83.207626) (end 113.10928 82.153056) (width 0.25) (layer B.Cu) (net 7))
   (segment (start 110.331216 83.207626) (end 112.05471 83.207626) (width 0.25) (layer B.Cu) (net 7))
-  (segment (start 112.384279 81.428055) (end 112.384279 61.879651) (width 0.25) (layer F.Cu) (net 7))
+  (segment (start 139.818944 54.173392) (end 143.509872 50.482464) (width 0.25) (layer F.Cu) (net 7))
+  (segment (start 118.42599 54.173392) (end 139.818944 54.173392) (width 0.25) (layer F.Cu) (net 7))
+  (segment (start 112.384279 60.215103) (end 118.42599 54.173392) (width 0.25) (layer F.Cu) (net 7))
+  (segment (start 112.384279 81.428055) (end 112.384279 60.215103) (width 0.25) (layer F.Cu) (net 7))
   (segment (start 113.10928 82.153056) (end 112.384279 81.428055) (width 0.25) (layer F.Cu) (net 7))
-  (segment (start 112.384279 61.879651) (end 121.876474 52.387456) (width 0.25) (layer F.Cu) (net 7))
-  (segment (start 127.912704 52.387456) (end 133.389568 46.910592) (width 0.25) (layer F.Cu) (net 7))
-  (segment (start 121.876474 52.387456) (end 127.912704 52.387456) (width 0.25) (layer F.Cu) (net 7))
   (segment (start 123.960714 79.907626) (end 129.381216 79.907626) (width 0.25) (layer B.Cu) (net 8))
   (segment (start 120.253024 76.199936) (end 123.960714 79.907626) (width 0.25) (layer B.Cu) (net 8))
@@
   (segment (start 112.054694 102.257626) (end 113.10928 101.20304) (width 0.25) (layer B.Cu) (net 12))
   (segment (start 110.331216 102.257626) (end 112.054694 102.257626) (width 0.25) (layer B.Cu) (net 12))
-  (segment (start 111.93427 100.02803) (end 111.93427 61.69325) (width 0.25) (layer F.Cu) (net 12))
+  (segment (start 137.874256 53.57808) (end 140.969872 50.482464) (width 0.25) (layer F.Cu) (net 12))
+  (segment (start 118.384892 53.57808) (end 137.874256 53.57808) (width 0.25) (layer F.Cu) (net 12))
+  (segment (start 111.934269 60.028703) (end 118.384892 53.57808) (width 0.25) (layer F.Cu) (net 12))
+  (segment (start 111.93427 100.02803) (end 111.934269 60.028703) (width 0.25) (layer F.Cu) (net 12))
   (segment (start 113.10928 101.20304) (end 111.93427 100.02803) (width 0.25) (layer F.Cu) (net 12))
-  (segment (start 111.93427 61.69325) (end 121.690074 51.937446) (width 0.25) (layer F.Cu) (net 12))
-  (segment (start 125.822714 51.937446) (end 130.849568 46.910592) (width 0.25) (layer F.Cu) (net 12))
-  (segment (start 121.690074 51.937446) (end 125.822714 51.937446) (width 0.25) (layer F.Cu) (net 12))
   (segment (start 113.883716 98.067626) (end 116.701422 95.24992) (width 0.25) (layer B.Cu) (net 13))
   (segment (start 116.701422 95.24992) (end 120.253024 95.24992) (width 0.25) (layer B.Cu) (net 13))
@@
   (via (at 113.10928 119.657712) (size 0.8) (drill 0.4) (layers F.Cu B.Cu) (net 17))
   (segment (start 110.331216 121.307626) (end 111.459366 121.307626) (width 0.25) (layer B.Cu) (net 17))
+  (segment (start 135.929568 52.982768) (end 138.429872 50.482464) (width 0.25) (layer F.Cu) (net 17))
+  (segment (start 118.343794 52.982768) (end 135.929568 52.982768) (width 0.25) (layer F.Cu) (net 17))
+  (segment (start 111.323344 60.003218) (end 118.343794 52.982768) (width 0.25) (layer F.Cu) (net 17))
+  (segment (start 111.323344 117.871776) (end 111.323344 60.003218) (width 0.25) (layer F.Cu) (net 17))
   (segment (start 113.10928 119.657712) (end 111.323344 117.871776) (width 0.25) (layer F.Cu) (net 17))
-  (segment (start 111.323344 61.667766) (end 121.503674 51.487436) (width 0.25) (layer F.Cu) (net 17))
-  (segment (start 111.323344 117.871776) (end 111.323344 61.667766) (width 0.25) (layer F.Cu) (net 17))
-  (segment (start 123.732724 51.487436) (end 128.309568 46.910592) (width 0.25) (layer F.Cu) (net 17))
-  (segment (start 121.503674 51.487436) (end 123.732724 51.487436) (width 0.25) (layer F.Cu) (net 17))
   (segment (start 113.883716 117.117626) (end 116.701438 114.299904) (width 0.25) (layer B.Cu) (net 18))
   (segment (start 116.701438 114.299904) (end 120.253024 114.299904) (width 0.25) (layer B.Cu) (net 18))
@@
   (segment (start 108.346784 114.240694) (end 108.683716 114.577626) (width 0.25) (layer B.Cu) (net 21))
   (segment (start 108.346784 111.323344) (end 108.346784 114.240694) (width 0.25) (layer B.Cu) (net 21))
-  (segment (start 134.183328 51.196832) (end 138.469568 46.910592) (width 0.25) (layer B.Cu) (net 21))
-  (segment (start 114.895216 51.196832) (end 134.183328 51.196832) (width 0.25) (layer B.Cu) (net 21))
-  (segment (start 108.683716 57.408332) (end 114.895216 51.196832) (width 0.25) (layer B.Cu) (net 21))
   (segment (start 108.683716 57.427626) (end 108.683716 57.408332) (width 0.25) (layer B.Cu) (net 21))
+  (segment (start 148.589872 50.482464) (end 145.348954 53.723382) (width 0.25) (layer B.Cu) (net 21))
+  (segment (start 112.38796 53.723382) (end 108.683716 57.427626) (width 0.25) (layer B.Cu) (net 21))
+  (segment (start 145.348954 53.723382) (end 112.38796 53.723382) (width 0.25) (layer B.Cu) (net 21))
   (via (at 127.396768 59.5312) (size 0.8) (drill 0.4) (layers F.Cu B.Cu) (net 22))
   (segment (start 127.733716 59.194252) (end 127.396768 59.5312) (width 0.25) (layer B.Cu) (net 22))
@@
   (segment (start 127.396768 114.240678) (end 127.733716 114.577626) (width 0.25) (layer B.Cu) (net 22))
   (segment (start 127.396768 111.323344) (end 127.396768 114.240678) (width 0.25) (layer B.Cu) (net 22))
-  (segment (start 127.733716 57.427626) (end 127.733716 53.836444) (width 0.25) (layer B.Cu) (net 22))
-  (segment (start 136.273318 51.646842) (end 141.009568 46.910592) (width 0.25) (layer B.Cu) (net 22))
-  (segment (start 129.923318 51.646842) (end 136.273318 51.646842) (width 0.25) (layer B.Cu) (net 22))
-  (segment (start 127.733716 53.836444) (end 129.923318 51.646842) (width 0.25) (layer B.Cu) (net 22))
+  (segment (start 127.733716 57.427626) (end 130.98795 54.173392) (width 0.25) (layer B.Cu) (net 22))
+  (segment (start 147.438944 54.173392) (end 151.129872 50.482464) (width 0.25) (layer B.Cu) (net 22))
+  (segment (start 130.98795 54.173392) (end 147.438944 54.173392) (width 0.25) (layer B.Cu) (net 22))
   (via (at 146.446752 59.5312) (size 0.8) (drill 0.4) (layers F.Cu B.Cu) (net 23))
   (segment (start 146.783716 59.194236) (end 146.446752 59.5312) (width 0.25) (layer B.Cu) (net 23))
@@
   (segment (start 146.446752 114.240662) (end 146.783716 114.577626) (width 0.25) (layer B.Cu) (net 23))
   (segment (start 146.446752 111.323344) (end 146.446752 114.240662) (width 0.25) (layer B.Cu) (net 23))
-  (segment (start 146.783716 50.14474) (end 143.549568 46.910592) (width 0.25) (layer B.Cu) (net 23))
-  (segment (start 146.783716 57.427626) (end 146.783716 50.14474) (width 0.25) (layer B.Cu) (net 23))
+  (segment (start 146.783716 57.427626) (end 146.783716 57.4083) (width 0.25) (layer B.Cu) (net 23))
+  (segment (start 146.783716 57.427626) (end 149.145638 57.427626) (width 0.25) (layer B.Cu) (net 23))
+  (segment (start 153.669872 52.903392) (end 153.669872 50.482464) (width 0.25) (layer B.Cu) (net 23))
+  (segment (start 149.145638 57.427626) (end 153.669872 52.903392) (width 0.25) (layer B.Cu) (net 23))
   (segment (start 165.833716 59.19422) (end 165.496736 59.5312) (width 0.25) (layer B.Cu) (net 24))
   (via (at 165.496736 59.5312) (size 0.8) (drill 0.4) (layers F.Cu B.Cu) (net 24))
@@
   (segment (start 165.496736 111.323344) (end 165.496736 114.240646) (width 0.25) (layer B.Cu) (net 24))
   (segment (start 165.77441 57.427626) (end 165.833716 57.427626) (width 0.25) (layer B.Cu) (net 24))
-  (segment (start 159.543616 51.196832) (end 165.77441 57.427626) (width 0.25) (layer B.Cu) (net 24))
-  (segment (start 150.375808 51.196832) (end 159.543616 51.196832) (width 0.25) (layer B.Cu) (net 24))
-  (segment (start 146.089568 46.910592) (end 150.375808 51.196832) (width 0.25) (layer B.Cu) (net 24))
+  (segment (start 165.833716 57.427626) (end 165.833716 56.296308) (width 0.25) (layer B.Cu) (net 24))
+  (segment (start 165.833716 56.296308) (end 163.115488 53.57808) (width 0.25) (layer B.Cu) (net 24))
+  (segment (start 159.305488 53.57808) (end 156.209872 50.482464) (width 0.25) (layer B.Cu) (net 24))
+  (segment (start 163.115488 53.57808) (end 159.305488 53.57808) (width 0.25) (layer B.Cu) (net 24))
   (zone (net 25) (net_name GND) (layer F.Cu) (hatch edge 0.508)
     (connect_pads (clearance 0.508))

Commit message: final
Parts:
- added D17: D_Small, Diode_SMD:D_SOD-123, B.Cu at (106.6, 48.2)
- added OL1: OLED, kbd:OLED_v2, F.Cu at (119.1, 42.9)
- added SW1: Rotary_Encoder_Switch, Keebio-Parts:RotaryEncoder_EC11, F.Cu at (102.4, 42.3)
Connections:
- U1 pad 13: Net-(U1-Pad13) -> /col2
- U1 pad 14: Net-(U1-Pad14) -> /col3
- U1 pad 15: Net-(U1-Pad15) -> /colRotEnc
- U1 pad 19: Net-(U1-Pad19) -> /pinA
- U1 pad 20: Net-(U1-Pad20) -> /pinB
- U1 pad 21: Net-(U1-Pad21) -> /VCC
- U1 pad 5: /col3 -> /SCL
- U1 pad 6: /col2 -> /SDA
Routing:
- net /pinB: track 0.00 -> 75.9 mm
- net /pinA: track 0.00 -> 66.0 mm
- net /col2: track 70.2 -> 126.5 mm
- net /SDA: track 0.00 -> 48.6 mm
- net /colRotEnc: track 0.00 -> 47.5 mm
- net /VCC: track 0.00 -> 43.4 mm
- net /SCL: track 0.00 -> 40.8 mm
- net /col3: track 72.2 -> 107.1 mm
- net /row3: track 158.3 -> 171.5 mm, vias 1 -> 2
- net /rotEnc: track 0.00 -> 7.76 mm
